File: positional.kicad_sch (KiCad schematic)
At the start: 0 parts

Commit message: preliminary positional schematic
Parts:
- added C1, C2, C3: 100 nF, symbol Device:C
- added U3: ISM330DHCXTR, EasyEDA:LGA-14_L3.0-W2.5-P0.50-BR, symbol EasyEDA:ISM330DHCXTR
- added U4: MS561101BA03-50, EasyEDA:SENSORS-SMD_MS5611-01BA03, symbol EasyEDA:MS561101BA03-50
Connections:
- net +3V3: now also C1.1, C2.1, C3.1, U3.12 (CS), U3.5 (VDD_IO), U3.8 (VDD), U4.1 (VDD), U4.2 (PS)
- net GND: now also C1.2, C2.2, C3.2, U3.1 (SDO/SA0), U3.2 (SDX), U3.3 (SCX), U3.6 (GND), U3.7 (GND), U4.3 (GND), U4.4 (CSB)
- net I2C1.SCL: now also U3.13 (SCL), U4.8 (SCLK)
- net I2C1.SDA: now also U3.14 (SDA), U4.7 (SDI/SDA)
