File: Data.kicad_sch (KiCad schematic)
At the start: 0 parts

Commit message: pre-fetch commit
Parts:
- added C1: 10u, symbol Device:C
- added C2: 100n, symbol Device:C
- added J1: MEM2067-02-180-00-A, MEM20670218000A, symbol MEM2067-02-180-00-A:MEM2067-02-180-00-A
- added R1, R2: 51k, symbol Device:R
Connections:
- net +3V3: now also C1.1, C1.2, C2.1, C2.2, J1.MP1, J1.MP2, J1.MP3, J1.MP4, J1.P4 (VDD), J1.P6 (VSS), R1.1, R2.2
- net SPI1.MISO: now also J1.P7 (DAT0)
- net SPI1.MOSI: now also J1.P3 (CMD)
- net SPI1.SCK: now also J1.P5 (CLK)
- net SPI1_CS_MICROSD: now also J1.P2 (CD/DAT3)
- new net: J1.P1 (DAT2), R2.1
- new net: J1.P8 (DAT1), R1.2

Commit message: prefixes added
Parts:
- renumbered C1 to C301, C2 to C302, R1 to R301, R2 to R302
Changed lines of the file:
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@@
 		(in_pos_files yes)
 		(dnp no)
-		(property "Reference" "C2"
+		(property "Reference" "C302"
 			(at 150.368 91.44 0)
 			(show_name no)
@@
 			(project "HAB5-OBC"
 				(path "/8bfdc6b4-3580-4cad-aef7-df6abccc03e5/52b36e2f-dbc1-4900-a8e8-742abd2560fa"
-					(reference "C2")
+					(reference "C302")
 					(unit 1)
 				)
@@
 		(in_pos_files yes)
 		(dnp no)
-		(property "Reference" "C1"
+		(property "Reference" "C301"
 			(at 138.938 91.44 0)
 			(show_name no)
@@
 			(project "HAB5-OBC"
 				(path "/8bfdc6b4-3580-4cad-aef7-df6abccc03e5/52b36e2f-dbc1-4900-a8e8-742abd2560fa"
-					(reference "C1")
+					(reference "C301")
 					(unit 1)
 				)
@@
 		(in_pos_files yes)
 		(dnp no)
-		(property "Reference" "R2"
+		(property "Reference" "R302"
 			(at 110.49 65.278 90)
 			(show_name no)
@@
 			(project "HAB5-OBC"
 				(path "/8bfdc6b4-3580-4cad-aef7-df6abccc03e5/52b36e2f-dbc1-4900-a8e8-742abd2560fa"
-					(reference "R2")
+					(reference "R302")
 					(unit 1)
 				)
@@
 		(in_pos_files yes)
 		(dnp no)
-		(fields_autoplaced yes)
 		(property "Reference" "#PWR011"
 			(at 110.49 67.31 0)
@@
 		)
 		(property "Value" "+3V3"
-			(at 102.87 67.3101 90)
-			(show_name no)
-			(do_not_autoplace no)
-			(effects
-				(font
-					(size 1.27 1.27)
-				)
-				(justify left)
+			(at 100.838 67.31 90)
+			(show_name no)
+			(do_not_autoplace no)
+			(effects
+				(font
+					(size 1.27 1.27)
+				)
 			)
 		)
@@
 		(in_pos_files yes)
 		(dnp no)
-		(property "Reference" "R1"
+		(property "Reference" "R301"
 			(at 171.45 67.818 90)
 			(show_name no)
@@
 			(project "HAB5-OBC"
 				(path "/8bfdc6b4-3580-4cad-aef7-df6abccc03e5/52b36e2f-dbc1-4900-a8e8-742abd2560fa"
-					(reference "R1")
-					(unit 1)
-				)
+					(reference "R301")
+					(unit 1)
+				)

Commit message: small fix
Parts:
- renumbered J1 to J301
Changed lines of the file:
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@@
 		(dnp no)
 		(fields_autoplaced yes)
-		(property "Reference" "J1"
+		(property "Reference" "J301"
 			(at 140.97 59.69 0)
 			(show_name no)
@@
 			(project "HAB5-OBC"
 				(path "/8bfdc6b4-3580-4cad-aef7-df6abccc03e5/52b36e2f-dbc1-4900-a8e8-742abd2560fa"
-					(reference "J1")
+					(reference "J301")
 					(unit 1)
 				)

Commit message: Add W25Q128 NOR flash on SPI2
Parts:
- added C303: 100n, symbol Device:C
- added R303, R304: 10k, symbol Device:R
- added U301: W25Q128JVS, Package_SO:SOIC-8_5.3x5.3mm_P1.27mm, symbol Memory_Flash:W25Q128JVS
Connections:
- net +3V3: now also C303.1, C303.2, R303.1, R304.2, U301.4 (GND), U301.8 (VCC)
- net SPI2.MISO: now also U301.2 (DO/IO_{1})
- net SPI2.MOSI: now also U301.5 (DI/IO_{0})
- net SPI2.SCK: now also U301.6 (CLK)
- net SPI2_CS_NOR: now also R303.2, U301.1 (~{CS})
- new net: R304.1, U301.3 (~{WP}/IO_{2}), U301.7 (~{HOLD}/~{RESET}/IO_{3})

Commit message: change NOR footprint and update refs
Parts:
- removed U301: W25Q128JVS, Package_SO:SOIC-8_5.3x5.3mm_P1.27mm, symbol Memory_Flash:W25Q128JVS
- added U3: W25Q128JVSIQTR, EasyEDA:SOIC-8_L5.3-W5.3-P1.27-LS8.0-BL, symbol EasyEDA:W25Q128JVSIQTR
Connections:
- net +3V3: now also U3.4 (GND), U3.8 (VCC)
- net SPI2.MISO: now also U3.2 (DO)
- net SPI2.MOSI: now also U3.5 (DI)
- net SPI2.SCK: now also U3.6 (CLK)
- net SPI2_CS_NOR: now also U3.1 (~{CS})
- net at R304.1: now also U3.3 (IO2), U3.7 (IO3)
