File: power.kicad_sch (KiCad schematic)
At the start: 0 parts

Commit message: Power (#4)
* add P-FET and fuse for battery and bench

* Add I2C, INA228 + accessories, and other small changes

* Added extra text for clarity

* new smaller resistor symbol

* power2

Added LDO and MUX

* rearrange mux resistors and new power bypass

* fix power to use correct symbol

* revert kicad proj file

---------

Co-authored-by: LakisunR <120803592+LakisunR@users.noreply.github.com>
Co-authored-by: cam <99922057+git-cam@users.noreply.github.com>
Parts:
- added C401, C404, C405: 100nF, EasyEDA:C0603, symbol Device:C_Small
- added C402, C407: 1uF, EasyEDA:C0805, symbol Device:C_Small
- added C403: 4.7uF, EasyEDA:C1206, symbol Device:C_Small
- added C406: 10uF, EasyEDA:C0805, symbol Device:C_Small
- added F401, F402: 500mA, EasyEDA:F1206, symbol HAB5OBC:0466.500NRHF
- added J1: (no value), symbol Connector:Conn_01x02_Pin
- added J2, J3: (no value), Connector_PinHeader_2.54mm:PinHeader_1x02_P2.54mm_Vertical, symbol Connector:Conn_01x02_Pin
- added Q401, Q402: AO3401A, EasyEDA:SOT-23_L2.9-W1.3-P1.90-LS2.4-BR, symbol HAB5OBC:AO3401A
- added R401, R402: 10k, EasyEDA:R0603, symbol HAB5OBC:0603WAF1002T5E
- added R403: 100mOhm, EasyEDA:R2512, symbol EasyEDA:LR2512-2AR100F4
- added R404: 68k, EasyEDA:R0603, symbol HAB5OBC:0603WAF6802T5E
- added R405, R407, R408, R410: 100k, EasyEDA:R0603, symbol HAB5OBC:0603WAF1003T5E
- added R406, R409: 39k, EasyEDA:R0603, symbol HAB5OBC:0603WAF3902T5E
- added U401: INA228AIDGSR, EasyEDA:VSSOP-10_L3.0-W3.0-P0.50-LS4.9-BL, symbol EasyEDA:INA228AIDGSR
- added U402: LDL1117S33R, EasyEDA:SOT-223-4_L6.5-W3.5-P2.30-LS7.0-BR, symbol EasyEDA:LDL1117S33R
- added U403: TPS2121RUXR, EasyEDA:VQFN-HR-12_L2.5-W2.0-P0.50-BL, symbol EasyEDA:TPS2121RUXR
Connections:
- new net: R408.1, U403.10 (ILM)
- new net: C404.2, U403.11 (SS)
- new net: C407.2, F402.2, R405.2, R407.2, U403.2 (IN2)
- new net: R409.2, R410.1, U403.5 (OV1)
- new net: F401.1, Q401.2 (S)
- new net: F401.2, R403.1, U401.10 (IN+)
- new net: Q402.1 (G), R402.2
- new net: Q401.1 (G), R401.2
- new net: C402.2, R403.2, U401.8 (VBUS), U401.9 (IN–), U402.3 (VIN)
- new net: F402.1, Q402.2 (S)
- new net +3V3: C401.2, C405.1, C406.1, J3.2 (Pin_2), U401.6 (VS), U403.1 (OUT), U403.8 (OUT)
- new net Battery_IN+: J1.2 (Pin_2), Q401.3 (D)
- new net Bench_IN+: J2.2 (Pin_2), Q402.3 (D)
- new net CP2: R404.2, R405.1, U403.3 (CP2)
- new net GND: C401.1, C402.1, C403.1, C404.1, C405.2, C406.2, C407.1, J1.1 (Pin_1), J2.1 (Pin_1), J3.1 (Pin_1), R401.1, R402.1, R404.1, R406.1, R408.2, R409.1, U401.1 (A1), U401.2 (A0), U401.7 (GND), U402.1 (GND), U403.12 (GND), U403.6 (PR1), U403.9 (ST)
- new net I2C1.SCL: U401.5 (SCL)
- new net I2C1.SDA: U401.4 (SDA)
- new net LDO_OUT: C403.2, R410.2, U402.2 (VOUT), U402.4 (VOUT), U403.7 (IN1)
- new net OV2: R406.2, R407.1, U403.4 (OV2)
- no-connect marks 0 -> 1
Other:
- note added: "Fuse"
- note added: "P-FET"
- note added: "Power Bypass"
- note added: "Shunt"
