File: HAB5-OBC.kicad_sch (KiCad schematic)
At the start: 1 part, among them U1 STM32F411CEU6

Commit message: Mcu connections and setup (#5)
* MCU core functionality

* Interface Connections

* change value for real value

* added NC flags

* Changed I2C pull up resistors

---------

Co-authored-by: alexhermeling <alex@hermeling.org>
Parts:
- added C101, C111: 4.7uF, EasyEDA:C1206, symbol EasyEDA:1206B475K500NT
- added C101, C102: 15pF, EasyEDA:C0402, symbol EasyEDA:0402CG150J500NT
- added C103, C104, C105, C106, C108, C109: 100nF, EasyEDA:C0402, symbol EasyEDA:CL05B104KO5NNNC
- added C107: 1uF, EasyEDA:C0805, symbol EasyEDA:CL21B105KBFNNNE
- added J101, J102, J103, J104: Conn_01x01_Pin, symbol Connector:Conn_01x01_Pin
- added R101: 10k, EasyEDA:R0402, symbol EasyEDA:0402WGF1002TCE
- added R101, R102: 4.7k, EasyEDA:R0603, symbol EasyEDA:0603WAF4701T5E
- added SW101: (no value), EasyEDA:SW-SMD_L3.9-W3.0-P4.45, symbol EasyEDA:TS-1088-AR02016
- added X101: 5032 8M 12PF 20PPM 4P, EasyEDA:CRYSTAL-SMD_4P-L5.0-W3.2-BL_ECS, symbol EasyEDA:50328M12PF20PPM4P
- renumbered U1 to U101
Connections:
- net I2C1.SCL: now also R102.1
- net I2C1.SDA: now also R101.1
- net +3V3: now reaches U101.1 (VBAT)
- net +3V3: now also U101.24 (VDD), U101.36 (VDD), U101.48 (VDD), U101.9 (VDDA/VREF+), C104.1, C105.1, C106.1, C107.1, C108.1, C109.1, C111.1, R101.2, R102.2
- net Temperature/LMT84_OUT: now reaches U101.10 (PA0)
- net Temperature/NTC_MID: now reaches U101.11 (PA1)
- net at U101.12 (PA2): now also J101.1 (Pin_1)
- net at U101.13 (PA3): now also J102.1 (Pin_1)
- net Data Handling/SPI1_CS_MICROSD: now reaches U101.14 (PA4)
- net SPI1.SCK: now reaches U101.15 (PA5)
- net SPI1.MISO: now reaches U101.16 (PA6)
- net SPI1.MOSI: now reaches U101.17 (PA7)
- net LED5: now reaches U101.20 (PB2)
- net SPI2.SCK: now reaches U101.21 (PB10)
- net at U101.22 (VCAP1): now also C101.1
- net GND: now reaches U101.23 (VSS)
- net GND: now also U101.35 (VSS), U101.47 (VSS), U101.49 (PAD), U101.8 (VSSA/VREF-), C101.1, C101.2, C102.2, C103.2, C104.2, C105.2, C106.2, C107.2, C108.2, C109.2, C111.2, R101.2, SW101.2, X101.2 (GND), X101.4 (GND)
- net Data Handling/SPI2_CS_NOR: now reaches U101.25 (PB12)
- net LED4: now reaches U101.26 (PB13)
- net SPI2.MISO: now reaches U101.27 (PB14)
- net SPI2.MOSI: now reaches U101.28 (PB15)
- net LED3: now reaches U101.29 (PA8)
- net USART1.TX: now reaches U101.30 (PA9)
- net USART1.RX: now reaches U101.31 (PA10)
- net LED0: now reaches U101.32 (PA11)
- net LED1: now reaches U101.33 (PA12)
- net SWD.SWDIO: now reaches U101.34 (PA13)
- net SWD.SWCLK: now reaches U101.37 (PA14)
- net LED2: now reaches U101.38 (PA15)
- net at U101.40 (PB4): now also J104.1 (Pin_1)
- net at U101.41 (PB5): now also J103.1 (Pin_1)
- net at U101.44 (BOOT0): now also R101.1
- net LED6: now reaches U101.45 (PB8)
- net LED7: now reaches U101.46 (PB9)
- net at U101.5 (PH0-OSC_IN): now also C102.1, X101.1
- net at U101.6 (PH1-OSC_OUT): now also C101.2, X101.3
- net at U101.7 (NRST): now also C103.1, SW101.1
- no-connect marks 0 -> 3
Other:
- sheet Data Handling ports: added SPI1_CS_MICROSD, SPI1{SCK MISO MOSI}, SPI2_CS_NOR, SPI2{SCK MISO MOSI}; removed none
- sheet Debug and Expansion ports: added LED[0..7], SWD{SWDIO SWCLK}, USART1{TX RX}; removed none
- sheet Positional Sheet ports: added I2C1{SDA SCL}; removed none
- sheet Temperature ports: added LMT84_OUT, NTC_MID; removed none
